Commit message: feat: implement cube reinforcement learning environment, add training/testing scripts, and update ignore rules

File: assets/cube.urdf (robot description, URDF)
Before this commit: robot balancing_cube, 3 links, 2 joints
Joints:
- joint motor: origin xyz=0 0 0.05 rpy=0 0 0 -> xyz=0 0 0.0707 rpy=0 0 0

Commit message: feat: add cube environment and URDF asset for reinforcement learning simulation

File: assets/cube.urdf (robot description, URDF)
Before this commit: robot balancing_cube, 3 links, 2 joints
Links:
- link cube_body: mass 0.5 -> 0.3
- link reaction_wheel: mass 0.1 -> 0.08; geometry visual cylinder length=0.01 radius=0.04
Joints:
- joint motor: limit effort=1.0 velocity=100.0 -> effort=1.0 velocity=400.0
